Commit message: Gazebo

File: project_arm_description/urdf/project_arm.xacro (robot description, xacro)
@@ -4,4 +4,10 @@
 <xacro:include filename="$(find project_arm_description)/urdf/project_arm.trans" />
 <xacro:include filename="$(find project_arm_description)/urdf/project_arm.gazebo" />
+<link name="world"/>
+  <joint name="world_joint" type="fixed">
+    <parent link="world"/>
+    <child link="base_link"/>
+    <origin xyz="0 0 0" rpy="0 0 0"/>
+  </joint>
 <link name="base_link">
   <inertial>

Commit message: Control Dinamico

File: project_arm_description/urdf/project_arm.xacro (robot description, xacro)
@@ -175,5 +175,5 @@
   <child link="link_1_1"/>
   <axis xyz="0.0 0.0 1.0"/>
-  <limit upper="3.141593" lower="0.0" effort="100" velocity="100"/>
+  <limit upper="3.141593" lower="0.0" effort="1000" velocity="10"/>
 </joint>
 <joint name="joint_2" type="revolute">
@@ -182,5 +182,5 @@
   <child link="link_2_1"/>
   <axis xyz="0.0 1.0 0.0"/>
-  <limit upper="1.570796" lower="-1.570796" effort="100" velocity="100"/>
+  <limit upper="1.570796" lower="-1.570796" effort="1000" velocity="10"/>
 </joint>
 <joint name="joint_3" type="revolute">
@@ -189,5 +189,5 @@
   <child link="link_3_1"/>
   <axis xyz="0.0 1.0 0.0"/>
-  <limit upper="0.785398" lower="-3.926991" effort="100" velocity="100"/>
+  <limit upper="0.785398" lower="-3.926991" effort="1000" velocity="10"/>
 </joint>
 <joint name="joint_4" type="revolute">
@@ -196,5 +196,5 @@
   <child link="link_4_1"/>
   <axis xyz="1.0 0.0 0.0"/>
-  <limit upper="3.141593" lower="0.0" effort="100" velocity="100"/>
+  <limit upper="3.141593" lower="0.0" effort="1000" velocity="10"/>
 </joint>
 <joint name="joint_5" type="revolute">
@@ -203,5 +203,5 @@
   <child link="link_5_1"/>
   <axis xyz="0.0 1.0 0.0"/>
-  <limit upper="2.356194" lower="-2.356194" effort="100" velocity="100"/>
+  <limit upper="2.356194" lower="-2.356194" effort="1000" velocity="10"/>
 </joint>
 <joint name="joint_6" type="revolute">
@@ -210,5 +210,5 @@
   <child link="link_6_1"/>
   <axis xyz="1.0 0.0 0.0"/>
-  <limit upper="6.283185" lower="0.0" effort="100" velocity="100"/>
+  <limit upper="6.283185" lower="0.0" effort="1000" velocity="10"/>
 </joint>
 <joint name="joint_7" type="prismatic">
@@ -217,5 +217,5 @@
   <child link="link_7_1"/>
   <axis xyz="1.0 0.0 0.0"/>
-  <limit upper="0.05" lower="0.0" effort="100" velocity="100"/>
+  <limit upper="0.05" lower="0.0" effort="1000" velocity="10"/>
 </joint>
 </robot>
